Commit message: Add a wrist camera for vision
Arducam UB0234 (1080p USB, 105 deg M12 lens) in a printed cradle on the
gripper's -y rail, tilted 15 deg toward the tool axis, with a 5 V LED light.
New docs/VISION.md covers the build, the cable splice, focusing, lens and
hand-eye calibration, AprilTag registration and the unload loop. The URDF
gains a wrist_camera_optical frame; BOM +$47 (bought parts $539).

Co-Authored-By: Claude Opus 5.5 <noreply@anthropic.com>
Claude-Session: https://claude.ai/code/session_01HFwANWvAhS26jNgU7RfycN

File: urdf/grip.urdf (robot description, URDF)
Before this commit: robot grip, 9 links, 8 joints
Links:
- added link wrist_camera_optical
- link tool: mass 0.2359 -> 0.2572
Joints:
- added joint wrist_camera: type fixed, parent tool, child wrist_camera_optical, origin xyz=0 -0.055 0.054 rpy=-0.26180 0 0
